File: PCB/GameTiger/GameTiger.kicad_sch (KiCad schematic)
At the start: 73 parts, among them J1 USB_C_Receptacle_USB2.0, J2 503398-1892, J3 LCD Display, J4 Speaker, Q3 DMG3415, U1 RP2040, U2 MCP73831-2-OT, U3 W25Q128JVSIQ, U4 PAM8302A, U5 AP2112K-3.3, U6 PCF8574TS, Y1 ABLS-12MHZ-B4-T

Commit message: Ready for uploading to JLCPCB
Parts:
- A1, B1, Down1, Left1, Right1, Up1: LCSC (none) -> C411882
- Boot1, Reset1: LCSC (none) -> C231329
- C1, C19, C22, C23, C4: LCSC (none) -> C1713
- C17, C18, C6, C9: LCSC (none) -> C14445
- C20, C21: LCSC (none) -> C61747
- D1: LCSC (none) -> C3018524
- D2: LCSC (none) -> C965791
- FB1, FB2: LCSC (none) -> C44838; Manuf. Part # BLM21AG102BH1D -> CBW201209U102T; Manufacturer Murata Electronics -> FH (Guangdong Fenghua Advanced Tech)
- J1: LCSC (none) -> C2988369
- J2: LCSC (none) -> C428492
- J3: LCSC (none) -> C262664; Manuf. Part # AFC07-S15FCA-00 -> AFC01-S15FCA-00
- Power1: LCSC (none) -> C221660
- Q3: LCSC (none) -> C96616
- R1, R5: LCSC (none) -> C11702
- R10, R12, R13, R16, R2, R6: LCSC (none) -> C25744
- R11, R14, R15: LCSC (none) -> C25905
- R3, R4: footprint Resistor_SMD:R_0402_1005Metric -> Resistor_SMD:R_0603_1608Metric; LCSC (none) -> C25190; Size 0402_1005Metric -> 0603_1608Metric
- R7: LCSC (none) -> C719176
- R8, R9: LCSC (none) -> C25076
- Select1, Start1: LCSC (none) -> C221678
- U1: LCSC (none) -> C2040
- U2: LCSC (none) -> C424093
- U3: LCSC (none) -> C113767
- U4: LCSC (none) -> C113367
- U5: LCSC (none) -> C51118
- U6: footprint Package_SO:SSOP-20_4.4x6.5mm_P0.65mm -> SOP65P640X150-20N; symbol Interface_Expansion:PCF8574TS -> PCF8574TS:PCF8574TS; A1_MIN (none) -> 0.0; A_MAX (none) -> 1.5; A_MIN (none) -> 1.5; A_NOM (none) -> 1.5; B_MAX (none) -> 0.32; B_MIN (none) -> 0.2; B_NOM (none) -> 0.26; D2_MAX (none) -> 0.0; D_MAX (none) -> 6.6; D_MIN (none) -> 6.4; D_NOM (none) -> 6.5; E1_MAX (none) -> 4.5; E1_MIN (none) -> 4.3; E1_NOM (none) -> 4.4; E2_MAX (none) -> 0.0; ENOM (none) -> 0.65; E_MAX (none) -> 6.6; E_MIN (none) -> 6.2; E_NOM (none) -> 6.4; LCSC (none) -> C57790; L_MAX (none) -> 0.75; L_MIN (none) -> 0.45; L_NOM (none) -> 0.6; MANUFACTURER (none) -> NXP; PARTREV (none) -> 5; PIN_COUNT (none) -> 20.0; STANDARD (none) -> IPC 7351B
- X1: LCSC (none) -> C295747
- Y1: LCSC (none) -> C2901718
Connections:
- net at U6.13 (NC): now also U6.18 (NC), U6.3 (NC), U6.8 (NC)
Other:
- moved on the sheet: J3

Commit message: Added battery level and charge detect connectors
Parts:
- added R17, R18: 100K, Resistor_SMD:R_0603_1608Metric, symbol Device:R_Small
- added R19: 5k6, Resistor_SMD:R_0603_1608Metric, symbol Device:R_Small
- added R20: 10K, Resistor_SMD:R_0603_1608Metric, symbol Device:R_Small
- C1, C19, C22, C23, C4: LCSC C1713 -> C15850; Material X5R -> (none); Tolerance 10% -> (none); Voltage 16v -> (none)
- C10, C11, C12, C13, C14, C15, C16, C5, C7, C8: LCSC (none) -> C1525; Material X7R -> (none); Tolerance 10% -> (none); Voltage 25v -> (none)
- C17, C18, C6, C9: LCSC C14445 -> C52923; Material X6S -> (none); Tolerance 10% -> (none); Voltage 10V -> (none)
- C2, C3: value 27pF -> 30pF; LCSC (none) -> C1570
- C20, C21: LCSC C61747 -> C107145; Material C0G -> (none); Tolerance 5% -> (none); Voltage 50v -> (none)
- D1: LCSC C3018524 -> C116159; Manuf. Part # MBR0540T1G -> MBR0540; Manufacturer FUXINSEMI -> Shikues
- J1: value USB_C_Receptacle_USB2.0 -> USB TypeC Connector; LCSC C2988369 -> C165948; Manuf. Part # GT-USB-7010ASV -> TYPE-C-31-M-12; Manufacturer G-Switch -> Korean Hroparts Elec
- Select1, Start1: footprint Button_Switch_SMD:SW_Push_1P1T_NO_CK_KMR2 -> Button_Switch_SMD:SW_SPST_Omron_B3FS-105xP; LCSC C221678 -> C306879; Manufacturer C&K -> Omron Electronics; Mfr.Part # KMR223GLFG -> B3FS-1052P
- U3: LCSC C113767 -> C97521
- U4: footprint PAM8302A:PAM8302A -> Package_SO:MSOP-8_3x3mm_P0.65mm
- U6: A1_MIN 0.0 -> (none); A_MAX 1.5 -> (none); A_MIN 1.5 -> (none); A_NOM 1.5 -> (none); B_MAX 0.32 -> (none); B_MIN 0.2 -> (none); B_NOM 0.26 -> (none); D2_MAX 0.0 -> (none); D_MAX 6.6 -> (none); D_MIN 6.4 -> (none); D_NOM 6.5 -> (none); E1_MAX 4.5 -> (none); E1_MIN 4.3 -> (none); E1_NOM 4.4 -> (none); E2_MAX 0.0 -> (none); ENOM 0.65 -> (none); E_MAX 6.6 -> (none); E_MIN 6.2 -> (none); E_NOM 6.4 -> (none); L_MAX 0.75 -> (none); L_MIN 0.45 -> (none); L_NOM 0.6 -> (none); MANUFACTURER NXP -> (none); PARTREV 5 -> (none); PIN_COUNT 20.0 -> (none); STANDARD IPC 7351B -> (none)
- Y1: value ABLS-12MHZ-B4-T -> 12MHZ XTal; footprint Crystal:Crystal_SMD_2520-4Pin_2.5x2.0mm -> Crystal:Crystal_SMD_3225-4Pin_3.2x2.5mm; LCSC C2901718 -> C9002; Manuf. Part # SX2B12.000F1210F30 -> X322512MSB4SI; Manufacturer Shenzhen SCTF Elec -> Yangxing Tech; Size SMD2520-4P -> SMD3225-4P
Connections:
- net GND: now also R18.1, R20.1
- net KYBD_INT: now also U1.28 (GPIO17); no longer U1.31 (GPIO20)
- net SX1262_BUSY: now also U1.14 (GPIO11); no longer U1.15 (GPIO12)
- net SX1262_CLK: now also U1.17 (GPIO14); no longer U1.18 (GPIO15)
- net SX1262_CS: now also U1.16 (GPIO13); no longer U1.17 (GPIO14)
- net SX1262_DIO1: now also U1.13 (GPIO10); no longer U1.14 (GPIO11)
- net SX1262_MISO: now also U1.15 (GPIO12); no longer U1.16 (GPIO13)
- net SX1262_MOSI: now also U1.18 (GPIO15); no longer U1.27 (GPIO16)
- net SX1262_RESET: now also U1.12 (GPIO9); no longer U1.28 (GPIO17)
- net VBAT: now also R17.1
- net VBUS: now also R19.1
- net BATTERY_LVL: now reaches U1.38 (GPIO26_ADC0)
- net BATTERY_LVL: now also R17.2, R18.2
- net POWER_USB_DM renamed POWER_USB_DN
- new net POWER_DETECT: R19.2, R20.2, U1.27 (GPIO16)
Other:
- note added: "Battery Level & Charging Detect"

Commit message: Completed updating the PCB design for peer review
Parts:
- removed R14, R15: 5.1K, Resistor_SMD:R_0402_1005Metric, symbol Device:R_Small
- removed Y1: 12MHZ XTal, Crystal:Crystal_SMD_3225-4Pin_3.2x2.5mm, symbol Device:Crystal_Small
- added R21, R22: 5.1K, Resistor_SMD:R_0402_1005Metric, symbol Device:R_Small
- added Y1: 12MHZ XTal, Crystal:Crystal_SMD_3225-4Pin_3.2x2.5mm, symbol Device:Crystal_GND24_Small
- A1, B1, Down1, Left1, Right1, Up1: footprint Button_Switch_SMD:SW_Push_1P1T_NO_CK_PTS125Sx43PSMTR -> Button_Switch_THT:SW_PUSH-12mm; Manufacturer C&K -> (none); Mfr.Part # PTS125SJM73PSMTR2LFS -> (none); Mouser (none) -> 653-B3F-1052; Size SMD,12x12mm -> (none)
- AE1: footprint Connector_Pin:Pin_D1.0mm_L10.0mm -> Connector_Pin:Pin_D1.0mm_L10.0mm_LooseFit
- Boot1, Reset1: Mouser (none) -> 653-B3U-1000P
- C1, C19, C22, C23, C4: Mouser (none) -> 187-CL21A106KAFN3NE; Size 0805_2012Metric -> (none)
- C10, C11, C12, C13, C14, C15, C16, C5, C7, C8: Mouser (none) -> 187-CL05A104KO5NNWC; Size 0402_1005Metric -> (none)
- C17, C18, C6, C9: Mouser (none) -> 187-CL05A105KP5NNWC; Size 0402_1005Metric -> (none)
- C2, C3: Material C0G -> (none); Size 0402_1005Metric -> (none); Tolerance 5% -> (none); Voltage 50v -> (none)
- C20, C21: Mouser (none) -> 187-CL21C221JB61PNL; Size 0805_2012Metric -> (none)
- D1: Mouser (none) -> 512-MBR0540
- D2: Mouser (none) -> 78-VLMO1500-GS08
- FB1, FB2: LCSC C44838 -> C85835; Manuf. Part # CBW201209U102T -> BLM21BD102SN1D; Manufacturer FH (Guangdong Fenghua Advanced Tech) -> Murata Electronics; Mouser (none) -> 81-BLM21B102S; Size 0805 -> (none)
- J1: LCSC C165948 -> C2988369; Manuf. Part # TYPE-C-31-M-12 -> GT-USB-7010ASV; Manufacturer Korean Hroparts Elec -> JAE Electronics; Mouser (none) -> 656-DX07S016JA1R1500
- J2: Mouser (none) -> 538-503398-1892
- J3: LCSC C262664 -> C262209; Manuf. Part # AFC01-S15FCA-00 -> 1-1734839-5; Manufacturer JUSHUO -> (none); Mouser (none) -> 571-1-1734839-5; Size SMD,P=0.5mm -> (none)
- Power1: Mouser (none) -> 611-JS102011SAQN; Size SMD -> (none)
- Q3: Mouser (none) -> 621-DMG3415U-7
- R1, R5: Mouser (none) -> 71-CRCW04021K00FKEDC; Power 63mW -> (none); Size 0402_1005Metric -> (none)
- R10, R12, R13, R16, R2, R6: Mouser (none) -> 71-CRCW040210K0FKEDC; Power 63mW -> (none); Size 0402_1005Metric -> (none)
- R11: Mouser (none) -> 71-CRCW04025K10FKEDC; Power 63mW -> (none); Size 0402_1005Metric -> (none)
- R17, R18: footprint Resistor_SMD:R_0603_1608Metric -> Resistor_SMD:R_0402_1005Metric; LCSC C25803 -> C25741; Mouser (none) -> 71-CRCW0402100KFKEDC; Size 0603_1608Metric -> (none)
- R19: footprint Resistor_SMD:R_0603_1608Metric -> Resistor_SMD:R_0402_1005Metric; LCSC (none) -> C25908; Mouser (none) -> 71-CRCW04025K60FKEDC; Size 0603_1608Metric -> (none)
- R20: footprint Resistor_SMD:R_0603_1608Metric -> Resistor_SMD:R_0402_1005Metric; LCSC (none) -> C25744; Mouser (none) -> 71-CRCW040210K0FKEDC; Size 0603_1608Metric -> (none)
- R3, R4: footprint Resistor_SMD:R_0603_1608Metric -> Resistor_SMD:R_0402_1005Metric; Mouser (none) -> 71-CRCW040227R0FKEDC; Power 63mW -> (none); Size 0603_1608Metric -> (none)
- R7: Mouser (none) -> 652-TC33X-2-103E
- R8, R9: Mouser (none) -> 71-CRCW0402100RFKEDC; Power 63mW -> (none); Size 0402_1005Metric -> (none)
- Select1, Start1: footprint Button_Switch_SMD:SW_SPST_Omron_B3FS-105xP -> Button_Switch_THT:SW_TH_Tactile_Omron_B3F-10xx; LCSC C306879 -> C411882; Manufacturer Omron Electronics -> (none); Mfr.Part # B3FS-1052P -> (none); Mouser (none) -> 653-B3F-1052; Size SMD -> SMD,6x6mm
- U1: Mouser (none) -> 358-SC091413
- U2: Mouser (none) -> 579-MCP73831T-2ACIOT
- U3: Mouser (none) -> 454-W25Q128JVSIQ
- U4: Mouser (none) -> 621-PAM8302AASCR
- U5: Mouser (none) -> 621-AP2112K-3.3TRG1
- U6: Manuf. Part # PCF8574TS -> PCF8574TS/3,118; Mouser (none) -> 771-PCF8574TDK-T
Connections:
- net BATTERY_LVL: now also R18.1; no longer R18.2
- net Crystal_XIN: now also Y1.1
- net Crystal_XOUT: now also Y1.3
- net GND: now also R18.2, R21.2, R22.2, Y1.2, Y1.4; no longer R18.1
- net at J1.B5 (CC2): now also R21.1
- net at J1.A5 (CC1): now also R22.1
Other:
- note added: "Battery Level & Charging"
- note removed: "Battery Level & Charging Detect"
- moved on the sheet: Boot1, C10, C11, C12, C13, C14, C15, C16, C2, C20, C21, C3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
