File: PCB/GameTiger/GameTiger.kicad_sch (KiCad schematic)
At the start: 77 parts, among them J1 USB TypeC Connector, J2 503398-1892, J3 LCD Display, J4 Speaker, Q3 DMG3415, U1 RP2040, U2 MCP73831-2-OT, U3 W25Q128JVSIQ, U4 PAM8302A, U5 AP2112K-3.3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

Commit message: Fixed differential pairs for USB-C connection
Parts:
- U3: footprint Package_SO:SOIC-8_5.23x5.23mm_P1.27mm -> Package_SO:SOP-8_5.28x5.23mm_P1.27mm; Size SOIC-8 208-mil -> SOP-8-208mil
Changed lines of the file:
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@@
       (effects (font (size 1.27 1.27)) (justify left))
     )
-    (property "Footprint" "Package_SO:SOIC-8_5.23x5.23mm_P1.27mm" (at 177.8 91.44 0)
+    (property "Footprint" "Package_SO:SOP-8_5.28x5.23mm_P1.27mm" (at 177.8 91.44 0)
       (effects (font (size 1.27 1.27)) hide)
     )
@@
       (effects (font (size 1.27 1.27)) hide)
     )
-    (property "Size" "SOIC-8 208-mil" (at 177.8 91.44 0)
+    (property "Size" "SOP-8-208mil" (at 177.8 91.44 0)
       (effects (font (size 1.27 1.27)) hide)
     )
@@
       (effects (font (size 1.27 1.27)) hide)
     )
-    (property "Datasheet" "https://datasheet.lcsc.com/lcsc/2008271404_BOURNS-TC33X-2-103E_C719176.pdf" (at 147.32 198.12 0)
-      (effects (font (size 1.27 1.27)) hide)
-    )
+    (property "Datasheet" "~" (at 147.32 198.12 0)
+      (effects (font (size 1.27 1.27)) hide)
+    )

Commit message: Redesigned pcb layout to fix errors in decoupling caps and ground plane
Parts:
- removed AE1: Antenna, Connector_Pin:Pin_D1.0mm_L10.0mm_LooseFit, symbol Device:Antenna
- removed U6: PCF8574TS, SOP65P640X150-20N, symbol PCF8574TS:PCF8574TS
- removed U7: ~, Waveshare:Core SX1262, symbol Waveshare:Core-SX1262
- U3: value W25Q128JVSIQ -> W25Q64JVSSIQ; footprint Package_SO:SOP-8_5.28x5.23mm_P1.27mm -> Package_SO:SOIC-8_5.23x5.23mm_P1.27mm; LCSC C97521 -> C179171; Manuf. Part # W25Q128JVSIQ -> W25Q64JVSSIQ; Mouser 454-W25Q128JVSIQ -> (none); Size SOP-8-208mil -> SOIC-8_5.23x5.23mm_P1.27mm
Connections:
- net KYBD_INT is gone; now on net KYBD_UP: U1.28 (GPIO17)
- net KYBD_SCL is gone; now on net KYBD_LEFT: U1.30 (GPIO19)
- net KYBD_SDA is gone; now on net KYBD_RIGHT: U1.29 (GPIO18)
- net SX1262_RESET is gone; now on net KYBD_SELECT: U1.12 (GPIO9)
- net Audio_PWM: now also U1.7 (GPIO5); no longer U1.8 (GPIO6)
- net GND: now also U1.19 (TESTEN)
- net KYBD_A: now also U1.8 (GPIO6)
- net KYBD_B: now also U1.9 (GPIO7)
- net KYBD_DOWN: now also U1.31 (GPIO20)
- net KYBD_START: now also U1.11 (GPIO8)
- net SX1262_BUSY: no longer names the net of U1.14 (GPIO11)
- net SX1262_CLK: no longer names the net of U1.17 (GPIO14)
- net SX1262_CS: no longer names the net of U1.16 (GPIO13)
- net SX1262_DIO1: no longer names the net of U1.13 (GPIO10)
- net SX1262_MISO: no longer names the net of U1.15 (GPIO12)
- net SX1262_MOSI: no longer names the net of U1.18 (GPIO15)
- no-connect marks 5 -> 2
Other:
- note removed: "8-Bit I/O Expander"
- note removed: "Core SX1262"
- moved on the sheet: J1, R21, R22

Commit message: PCB Design track cleanup
Parts:
- removed H1, H2, H3, H4: MountingHole, MountingHole:MountingHole_2.2mm_M2, symbol Mechanical:MountingHole
- A1: value SW_Push -> A
- B1: value SW_Push -> B
- Boot1: value SW_Push -> Boot
- Down1: value SW_Push -> Down
- Left1: value SW_Push -> Left
- Power1: value SW_Push -> Power
- Reset1: value SW_Push -> Reset
- Right1: value SW_Push -> Right
- Select1: value SW_Push -> Select
- Start1: value SW_Push -> Start
- Up1: value SW_Push -> Up
Other:
- note removed: "PCB Mounting Holes"

Commit message: Minor fixes in PCB design
Parts:
- added FID1, FID2, FID3: ~, Fiducial:Fiducial_1mm_Mask2mm, symbol GameTiger-eagle-import:FIDUCIAL_1MM
Changed lines of the file:
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@@
+    )
+  )
+  (symbol (lib_id "GameTiger-eagle-import:FIDUCIAL_1MM") (at 245.11 266.7 0) (unit 1)
+    (in_bom yes) (on_board yes) (dnp no) (fields_autoplaced)
+    (property "Reference" "FID1" (at 245.11 266.7 0)
+      (effects (font (size 1.27 1.27)) hide)
+    )
+    (property "Value" "~" (at 245.11 266.7 0)
+      (effects (font (size 1.27 1.27)) hide)
+    )
+    (property "Footprint" "Fiducial:Fiducial_1mm_Mask2mm" (at 245.11 266.7 0)
+      (effects (font (size 1.27 1.27)) hide)
+    )
+    (property "Datasheet" "" (at 245.11 266.7 0)
+      (effects (font (size 1.27 1.27)) hide)
+    )
+    (instances
+      (project "GameTiger"
+        (path "/c33a9324-58b6-4ca3-8378-bbd431fb85f4"
+          (reference "FID1") (unit 1)
+        )
+      )
     )
   )
@@
         (path "/c33a9324-58b6-4ca3-8378-bbd431fb85f4"
           (reference "#PWR05") (unit 1)
+        )
+      )
+    )
+  )
+  (symbol (lib_id "GameTiger-eagle-import:FIDUCIAL_1MM") (at 250.19 266.7 0) (unit 1)
+    (in_bom yes) (on_board yes) (dnp no) (fields_autoplaced)
+    (property "Reference" "FID2" (at 250.19 266.7 0)
+      (effects (font (size 1.27 1.27)) hide)
+    )
+    (property "Value" "~" (at 250.19 266.7 0)
+      (effects (font (size 1.27 1.27)) hide)
+    )
+    (property "Footprint" "Fiducial:Fiducial_1mm_Mask2mm" (at 250.19 266.7 0)
+      (effects (font (size 1.27 1.27)) hide)
+    )
+    (property "Datasheet" "" (at 250.19 266.7 0)
+      (effects (font (size 1.27 1.27)) hide)
+    )
+    (instances
+      (project "GameTiger"
+        (path "/c33a9324-58b6-4ca3-8378-bbd431fb85f4"
+          (reference "FID2") (unit 1)
         )
       )
@@
         )
       )
+    )
+  )
+  (symbol (lib_id "GameTiger-eagle-import:FIDUCIAL_1MM") (at 255.27 266.7 0) (unit 1)
+    (in_bom yes) (on_board yes) (dnp no) (fields_autoplaced)
+    (property "Reference" "FID3" (at 255.27 266.7 0)
+      (effects (font (size 1.27 1.27)) hide)
+    )
+    (property "Value" "~" (at 255.27 266.7 0)
+      (effects (font (size 1.27 1.27)) hide)
+    )
+    (property "Footprint" "Fiducial:Fiducial_1mm_Mask2mm" (at 255.27 266.7 0)
+      (effects (font (size 1.27 1.27)) hide)
+    )
+    (property "Datasheet" "" (at 255.27 266.7 0)
+      (effects (font (size 1.27 1.27)) hide)
+    )
+    (instances
+      (project "GameTiger"
+        (path "/c33a9324-58b6-4ca3-8378-bbd431fb85f4"
+          (reference "FID3") (unit 1)
+        )
+      )

Commit message: PCB design completed and ordered for fab
Parts:
- removed FID1, FID2, FID3: ~, Fiducial:Fiducial_1mm_Mask2mm, symbol GameTiger-eagle-import:FIDUCIAL_1MM
- removed Power1: Power, Button_Switch_SMD:SW_SPDT_CK-JS102011SAQN, symbol Switch:SW_Push
- added J5: Conn_01x03, Connector_Wire:SolderWire-0.25sqmm_1x03_P4.2mm_D0.65mm_OD1.7mm, symbol Connector_Generic:Conn_01x03
- added Power1: Power, MK-12C02-G020:MK-12C02-G020_GSW, symbol MK-12C02-G020:MK-12C02-G020
- R2: now not fitted; now left out of the parts list
- U4: Mouser 621-PAM8302AASCR -> (none)
- U5: footprint Package_TO_SOT_SMD:SOT-23-5 -> AP2112K-3-3TRG1:SOT_RG1_DIO
Connections:
- net EN: now also Power1.1
- net GND: now also J5.2 (Pin_2), Power1.2
- net SW_CLK: now reaches U1.24 (SWCLK)
- net SW_CLK: now also J5.1 (Pin_1)
- net SW_DIO: now reaches U1.25 (SWD)
- net SW_DIO: now also J5.3 (Pin_3)
Other:
- note added: "Serial Wire Debug"
- moved on the sheet: X1A

Commit message: Added Blender file for 3D printing Case
Parts:
- A1, B1, Down1, Left1, Right1, Up1: footprint Button_Switch_THT:SW_PUSH-12mm -> Button_Switch_THT:SW_PUSH-12mm_3DModel
Changed lines of the file:
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@@
       (effects (font (size 1.27 1.27)))
     )
-    (property "Footprint" "Button_Switch_THT:SW_PUSH-12mm" (at 52.07 255.27 0)
+    (property "Footprint" "Button_Switch_THT:SW_PUSH-12mm_3DModel" (at 52.07 255.27 0)
       (effects (font (size 1.27 1.27)) hide)
     )
@@
       (effects (font (size 1.27 1.27)))
     )
-    (property "Footprint" "Button_Switch_THT:SW_PUSH-12mm" (at 66.04 252.73 0)
+    (property "Footprint" "Button_Switch_THT:SW_PUSH-12mm_3DModel" (at 66.04 252.73 0)
       (effects (font (size 1.27 1.27)) hide)
     )
@@
       (effects (font (size 1.27 1.27)))
     )
-    (property "Footprint" "Button_Switch_THT:SW_PUSH-12mm" (at 38.1 270.51 0)
+    (property "Footprint" "Button_Switch_THT:SW_PUSH-12mm_3DModel" (at 38.1 270.51 0)
       (effects (font (size 1.27 1.27)) hide)
     )
@@
       (effects (font (size 1.27 1.27)))
     )
-    (property "Footprint" "Button_Switch_THT:SW_PUSH-12mm" (at 52.07 273.05 0)
+    (property "Footprint" "Button_Switch_THT:SW_PUSH-12mm_3DModel" (at 52.07 273.05 0)
       (effects (font (size 1.27 1.27)) hide)
     )
@@
       (effects (font (size 1.27 1.27)))
     )
-    (property "Footprint" "Button_Switch_THT:SW_PUSH-12mm" (at 80.01 250.19 0)
+    (property "Footprint" "Button_Switch_THT:SW_PUSH-12mm_3DModel" (at 80.01 250.19 0)
       (effects (font (size 1.27 1.27)) hide)
     )
@@
       (effects (font (size 1.27 1.27)))
     )
-    (property "Footprint" "Button_Switch_THT:SW_PUSH-12mm" (at 38.1 257.81 0)
-      (effects (font (size 1.27 1.27)) hide)
-    )
+    (property "Footprint" "Button_Switch_THT:SW_PUSH-12mm_3DModel" (at 38.1 257.81 0)
+      (effects (font (size 1.27 1.27)) hide)
+    )
